Commit message: making changes to sensor. Rviz shows all points

File: urdf/hku_m100.urdf.xacro (robot description, xacro)
@@ -1,5 +1,5 @@
 <?xml version="1.0"?>
 <robot name="uav1" xmlns:xacro="http://www.ros.org/wiki/xacro">
-    <xacro:include filename="$(find hku_m100_description)/urdf/hku_m100_base_with_gimbal.urdf.xacro" />
+    <xacro:include filename="$(find hku_m100_gazebo)/urdf/hku_m100_base_with_gimbal.urdf.xacro" />
     <xacro:hku_m100_base_macro />
 </robot>

File: urdf/hku_m100_base_with_gimbal.urdf.xacro (robot description, xacro)
@@ -58,69 +58,8 @@
  -->
   <!-- <xacro:include filename="$(find hku_m100_description)/urdf/hku_m100.gazebo" /> -->
-<!--   <xacro:include filename="$(find hku_m100_description)/urdf/gimbal_camera.urdf.xacro"/>
+  <xacro:include filename="$(find hku_m100_description)/urdf/gimbal_camera.urdf.xacro"/>
   <xacro:gimbal_camera name="camera" parent="base_link" ros_topic="camera/image" cam_info_topic="camera/camera_info" update_rate="10" res_x="320" res_y="240" image_format="R8G8B8" hfov="90">
     <origin xyz="0.05 0.0 -0.06" rpy="0 0 0"/>
   </xacro:gimbal_camera>
- -->
-   <joint name="camera_joint" type="floating">
-      <origin xyz="0.1 0 -0.04" rpy="0 0 0"/>
-      <parent link="base_link"/>
-      <child link="camera_link"/>
-    </joint>
-    <link name="camera_link">
-      <inertial>
-        <mass value="0.0010" />
-        <origin xyz="0 0 0" rpy="0 0 0" />
-        <inertia ixx="0.0001" ixy="0" ixz="0" iyy="0.0001" iyz="0" izz="0.0001" />
-      </inertial>
-      <visual>
-        <origin xyz="0 0 0" rpy="0 0 0" />
-        <geometry>
-          <mesh filename="package://hku_m100_description/meshes/hku_m100/gimbal.dae"/>
-        </geometry>
-      </visual>
-      <collision>
-        <origin xyz="0 0 0" rpy="0 0 0" />
-        <geometry>
-          <mesh filename="package://hku_m100_description/meshes/hku_m100/gimbal.stl"/>
-        </geometry>
-      </collision>
-    </link>
-    <joint name="camera_optical_joint" type="floating">
-      <origin xyz="0 0 0" rpy="${-M_PI/2} 0.0 ${-M_PI/2}" />
-      <parent link="camera_link" />
-      <child link="camera_optical_frame"/>
-    </joint>
-    <link name="camera_optical_frame"/>
-    <gazebo reference="camera_link">
-      <sensor type="camera" name="camera_camera_sensor">
-        <update_rate>10</update_rate>
-        <camera>
-          <!-- <pose>0.027 0 -0.027 0 1.57 0</pose> -->
-          <!-- <pose>0.027 0 -0.027 0 1.57 0</pose> -->
-          <pose>0.027 0 -0.027 0 0 0</pose>
-          <horizontal_fov>${94 * M_PI/180.0}</horizontal_fov>
-          <image>
-            <format>R8G8B8</format>
-            <width>640</width>
-            <height>480</height>
-          </image>
-          <clip>
-            <near>0.01</near>
-            <far>100</far>
-          </clip>
-        </camera>
-        <plugin name="camera_controller" filename="libgazebo_ros_camera.so">
-          <cameraName>camera</cameraName>
-          <alwaysOn>true</alwaysOn>
-          <updateRate>10</updateRate>
-          <imageTopicName>/dji_sdk/image_raw</imageTopicName>
-          <cameraInfoTopicName>/dji_sdk/camera_info</cameraInfoTopicName>
-          <!-- <imageTopicName>camera/image</imageTopicName> -->
-          <!-- <cameraInfoTopicName>camera/camera_info</cameraInfoTopicName> -->
-          <frameName>camera_optical_frame</frameName>
-        </plugin>
-      </sensor>
-    </gazebo>
   </xacro:macro>
 </robot>
