Commit message: changed some of the configuration files

File: urdf/hku_m100_base.urdf.xacro (robot description, xacro)
@@ -13,5 +13,5 @@
         <origin xyz="0 0 0" rpy="0 0 0" />
         <geometry>
-          <mesh filename="package://hku_m100_description/meshes/hku_m100/hku_m100.dae"/>
+          <mesh filename="package://hku_m100_gazebo/meshes/hku_m100/hku_m100.dae"/>
         </geometry>
       </visual>
@@ -19,5 +19,5 @@
         <origin xyz="0 0 0" rpy="0 0 0" />
         <geometry>
-          <mesh filename="package://hku_m100_description/meshes/hku_m100/hku_m100.stl"/>
+          <mesh filename="package://hku_m100_gazebo/meshes/hku_m100/hku_m100.stl"/>
         </geometry>
       </collision>

File: urdf/hku_m100_base_with_gimbal.urdf.xacro (robot description, xacro)
@@ -16,5 +16,5 @@
         <origin xyz="0 0 0" rpy="0 0 0" />
         <geometry>
-          <mesh filename="package://hku_m100_description/meshes/hku_m100/hku_m100.dae"/>
+          <mesh filename="package://hku_m100_gazebo/meshes/hku_m100/hku_m100.dae"/>
         </geometry>
       </visual>
@@ -22,5 +22,5 @@
         <origin xyz="0 0 0" rpy="0 0 0" />
         <geometry>
-          <mesh filename="package://hku_m100_description/meshes/hku_m100/hku_m100.stl"/>
+          <mesh filename="package://hku_m100_gazebo/meshes/hku_m100/hku_m100.stl"/>
         </geometry>
       </collision>
@@ -58,5 +58,5 @@
  -->
   <!-- <xacro:include filename="$(find hku_m100_description)/urdf/hku_m100.gazebo" /> -->
-  <xacro:include filename="$(find hku_m100_description)/urdf/gimbal_camera.urdf.xacro"/>
+  <xacro:include filename="$(find hku_m100_gazebo)/urdf/gimbal_camera.urdf.xacro"/>
   <xacro:gimbal_camera name="camera" parent="base_link" ros_topic="camera/image" cam_info_topic="camera/camera_info" update_rate="10" res_x="320" res_y="240" image_format="R8G8B8" hfov="90">
     <origin xyz="0.05 0.0 -0.06" rpy="0 0 0"/>

Commit message: I am now sure, that rviz is running backwards

File: urdf/hku_m100_base.urdf.xacro (robot description, xacro)
@@ -7,5 +7,5 @@
       <inertial>
         <mass value="1.477" />
-        <origin xyz="0 0 0" />
+        <origin xyz="0 0 0" rpy="0 0 0"/>
         <inertia ixx="0.01152" ixy="0.0" ixz="0.0" iyy="0.01152" iyz="0.0" izz="0.0218" />
       </inertial>
