Commit message: just need to fix transform from baselink to world

File: urdf/hku_m100_base_with_gimbal.urdf.xacro (robot description, xacro)
@@ -1,5 +1,5 @@
 <?xml version="1.0"?>
 <robot xmlns:xacro="http://www.ros.org/wiki/xacro">
-  <xacro:property name="pi" value="3.1415926535897931" />
+  <!--<xacro:property name="pi" value="3.1415926535897931" />-->
   <xacro:property name="M_PI" value="3.1415926535897931" />
 <!--   <xacro:include filename="$(find hku_m100_description)/urdf/hku_m100.gazebo" />

Commit message: got it running, fixed map

File: urdf/hku_m100_base_with_gimbal.urdf.xacro (robot description, xacro)
@@ -10,5 +10,5 @@
       <inertial>
         <mass value="1.477" />
-        <origin xyz="0 0 0" />
+        <origin xyz="0 0 0" rpy="0 0 0"/>
         <inertia ixx="0.01152" ixy="0.0" ixz="0.0" iyy="0.01152" iyz="0.0" izz="0.0218" />
       </inertial>
